File: ESP32/Smart_Robotic_Car_With_PID_control/hardware/Smart_Robotic_Car_With_PID_control.kicad_sch (KiCad schematic)
At the start: 108 parts, among them J1 BSENS, J10 MOTOR 2, J11 MOTOR 4, J12 OUT+, J13 OUT-, J14 MPU6050, J15 UART, J16 I2C, J17 12V IN, J18 USB_C Conn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

Commit message: updated projects
Parts:
- JP1, JP2, JP5, JP6: value ~ -> (none)
