File: ESP32/Fingerprint_and_RFID_Card_Attendance_System/hardware/Fingerprint_and_RFID_Card_Attendance_System.kicad_sch (KiCad schematic)
At the start: 65 parts, among them J1 RTC, J10 -UPS, J11 V_OUT, J12 +BATT, J13 BUTTONS, J14 AS608, J15 SD MODULE, J16 -BATT, J17 SW_C, J18 SW_NO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

Commit message: updated projects
Parts:
- JP1, JP2, JP3: value ~ -> (none)
