File: ESP32/NFC_Card_Payment_System/hardware/NFC_Card_Payment_System.kicad_sch (KiCad schematic)
At the start: 63 parts, among them J1 RTC, J10 -UPS, J11 V_OUT, J12 +BATT, J13 BUTTONS, J15 SD MODULE, J16 -BATT, J17 SW_C, J18 SW_NO, J2 128X64 2.42 INCH OLED SCREEN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

Commit message: updated from work
Parts:
- JP1, JP2, JP3: value ~ -> (none)
Other:
- note added: "NFC CARD PAYMENT"
- note added: "SYSTEM"
- note removed: "AND"
- note removed: "ATTENDANCE SYSTEM"
- note removed: "FINGERPRINT"
- note removed: "RFID CARD"
