File: ESP32/Dual_Axis_Solar_Tracker/hardware/Dual_Axis_Solar_Tracker.kicad_sch (KiCad schematic)
At the start: 76 parts, among them J1 12VAC, J2 12VAC, J3 SIGNAL, J4 MOTOR, J5 12V_IN, J6 USB_C Conn, M1 Geared Motor, M2 Geared Motor, Q1 UMH3N, SW1 RotaryEncoder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

Commit message: update from home
Parts:
- JP1: value ~ -> (none)
