File: ESP32/Smart_Home_Energy_Management_System/hardware/Smart_Home_Energy_Management_System.kicad_sch (KiCad schematic)
At the start: 141 parts, among them J1 NEPA, J10 N, J11 PZEM_SIG, J14 USB_C Conn, J15 TRANS 1-OUT, J16 128X64 GLCD, J17 TRANS-IN, J18 TRANS 2-OUT, J19 DISPLAY, J2 INVERTER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

Commit message: update from home
Parts:
- JP1, JP2, JP3: value ~ -> (none)
