File: ESP32/Solar_Powered_Irrigation_System/hardware/Solar_Powered_Irrigation_System.kicad_sch (KiCad schematic)
At the start: 78 parts, among them J1 PUMP, J10 -BATT, J11 INPUT, J12 +BATT, J13 +5V, J14 -5V, J15 BSEN, J2 SOIL SENSOR, J3 AM2301A, J4 OLED SCREEN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

Commit message: update from home
Parts:
- JP1: value ~ -> (none)
