File: ESP32/Predictive_Maintenance_System_for_Industrial_Motor/hardware/_restore_backup_2026-06-09T05-09-15-000/Predictive_Maintenance_System_for_Industrial_Motor.kicad_sch (KiCad schematic)
At the start: 81 parts, among them J1 DS18B20, J2 CURRENT SENSOR, J3 OLED SCREEN, J4 LOAD, J5 220VAC, J6 MPU6050, J7 SD MODULE, J8 USB_C Conn, J9 12VAC, K1 FINDER-36.11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

Commit message: Updated project files
Parts:
- JP1: value (none) -> ~
